Commit message: SIMULATION: fix camera macro

File: simulation/navigator_gazebo/urdf/camera.xacro (robot description, xacro)
@@ -3,41 +3,9 @@
   <!-- Macro for inserting an engine with its propeller. -->
   <xacro:macro  name="navigator_camera"
-                params="name
+                params="name namespace:='/camera'
                         parent='base_link' xyz:='0 0 0' rpy:='0 0 0'
                         width:=960 height:=600 fov:=1.047 fps:=30
                         k1:=0 k2:=0 t1:=0 t2:=0 k3:=0">
-    <link name="${name}">
-      <gazebo>
-        <sensor name="${name}_sensor" type="camera">
-          <camera>
-            <pose>0 0 0 0 0 0</pose>
-            <horizontal_fov>1.047</horizontal_fov>
-            <image>
-              <width>960</width>
-              <height>600</height>
-            </image>
-            <distortion>
-              <k1>${k1}</k1>
-              <k2>${k2}</k2>
-              <k3>${k3}</k3>
-              <p1>${t1}</p1>
-              <p2>${t2}</p2>
-            </distortion>
-          </camera>
-          <plugin name="${name}_controller" filename="libgazebo_ros_camera.so">
-            <updateRate>${30}</updateRate>
-            <cameraName>${name}</cameraName>
-            <imageTopicName>image_raw</imageTopicName>
-            <cameraInfoTopicName>camera_info</cameraInfoTopicName>
-            <frameName>${name}_optical</frameName>
-            <distortionK1>${k1}</distortionK1>
-            <distortionK2>${k2}</distortionK2>
-            <distortionK3>${k3}</distortionK3>
-            <distortionT1>${t1}</distortionT1>
-            <distortionT2>${t2}</distortionT2>
-          </plugin>
-        </sensor>
-      </gazebo>
-    </link>
+    <link name="${name}" />
     <joint name="${name}_to_${parent}" type="fixed">
       <parent link="${parent}" />
@@ -51,4 +19,37 @@
       <origin xyz="0 0 0" rpy="${-pi/2} 0 ${-pi/2}"/>
     </joint>
+    <gazebo reference="${name}">
+      <sensor name="${name}_sensor" type="camera">
+        <update_rate>${fps}</update_rate>
+        <camera name="${name}_camera">
+          <pose>0 0 0 0 0 0</pose>
+          <horizontal_fov>1.047</horizontal_fov>
+          <image>
+            <width>960</width>
+            <height>600</height>
+          </image>
+          <distortion>
+            <k1>${k1}</k1>
+            <k2>${k2}</k2>
+            <k3>${k3}</k3>
+            <p1>${t1}</p1>
+            <p2>${t2}</p2>
+          </distortion>
+        </camera>
+        <plugin name="${name}_controller" filename="libgazebo_ros_camera.so">
+          <robotNamespace>${namespace}</robotNamespace>
+          <alwaysOn>true</alwaysOn>
+          <updateRate>0</updateRate>
+          <imageTopicName>image_raw</imageTopicName>
+          <cameraInfoTopicName>camera_info</cameraInfoTopicName>
+          <frameName>${name}_optical</frameName>
+          <distortionK1>${k1}</distortionK1>
+          <distortionK2>${k2}</distortionK2>
+          <distortionK3>${k3}</distortionK3>
+          <distortionT1>${t1}</distortionT1>
+          <distortionT2>${t2}</distortionT2>
+        </plugin>
+      </sensor>
+    </gazebo>
   </xacro:macro>
 </robot>

File: simulation/navigator_gazebo/urdf/navigator.urdf.xacro (robot description, xacro)
@@ -19,11 +19,11 @@
   <!-- Camera frames with gazebo simulation plugins -->
   <xacro:include filename="$(find navigator_gazebo)/urdf/camera.xacro" />
-  <xacro:navigator_camera name="front_left_cam" parent="velodyne"
+  <xacro:navigator_camera name="front_left_cam" parent="velodyne" namespace="/camera/front/left/"
                           xyz="0.294 0.1 -0.45"
                           rpy="0 0.258 0" />
-  <xacro:navigator_camera name="front_right_cam" parent="velodyne"
+  <xacro:navigator_camera name="front_right_cam" parent="velodyne" namespace="/camera/front/right/"
                           xyz="0.294 -0.099 -0.45"
                           rpy="0 0.258 0" />
-  <xacro:navigator_camera name="starboard_cam" parent="measurement"
+  <xacro:navigator_camera name="starboard_cam" parent="measurement" namespace="/camera/starboard/"
                           xyz="-0.285 -0.495 0.129"
                           rpy="0 0 -1.570796" />
